File: hardware/hexpansion.kicad_sch (KiCad schematic)
At the start: 95 parts, among them J1 Hexpansion-Connector, J2 Conn_01x03_Pin, SW1 SW_Push, SW2 SW_Push, U1 MT3608, U10 XL-0807RGBC-WS2812B-S, U11 XL-0807RGBC-WS2812B-S, U12 XL-0807RGBC-WS2812B-S, U13 XL-0807RGBC-WS2812B-S, U14 XL-0807RGBC-WS2812B-S, U15 XL-0807RGBC-WS2812B-S, U16 XL-0807RGBC-WS2812B-S, U17 XL-0807RGBC-WS2812B-S, U18 XL-0807RGBC-WS2812B-S, U19 XL-0807RGBC-WS2812B-S, U2 ZD24C64A-XGMT, U20 XL-0807RGBC-WS2812B-S, U21 XL-0807RGBC-WS2812B-S, U22 XL-0807RGBC-WS2812B-S, U23 XL-0807RGBC-WS2812B-S, U24 XL-0807RGBC-WS2812B-S, U25 XL-0807RGBC-WS2812B-S, U26 XL-0807RGBC-WS2812B-S, U27 XL-0807RGBC-WS2812B-S, U28 XL-0807RGBC-WS2812B-S, U29 XL-0807RGBC-WS2812B-S, U3 XL-0807RGBC-WS2812B-S, U30 XL-0807RGBC-WS2812B-S, U31 XL-0807RGBC-WS2812B-S, U32 XL-0807RGBC-WS2812B-S, U33 XL-0807RGBC-WS2812B-S, U34 XL-0807RGBC-WS2812B-S, U35 XL-0807RGBC-WS2812B-S, U36 XL-0807RGBC-WS2812B-S, U37 XL-0807RGBC-WS2812B-S, U38 XL-0807RGBC-WS2812B-S, U39 XL-0807RGBC-WS2812B-S, U4 XL-0807RGBC-WS2812B-S, U40 XL-0807RGBC-WS2812B-S, U41 XL-0807RGBC-WS2812B-S, U42 XL-0807RGBC-WS2812B-S, U43 XL-0807RGBC-WS2812B-S, U44 XL-0807RGBC-WS2812B-S, U45 XL-0807RGBC-WS2812B-S, U46 XL-0807RGBC-WS2812B-S, U47 XL-0807RGBC-WS2812B-S, U48 XL-0807RGBC-WS2812B-S, U49 XL-0807RGBC-WS2812B-S, U5 XL-0807RGBC-WS2812B-S, U50 XL-0807RGBC-WS2812B-S, U51 XL-0807RGBC-WS2812B-S, U52 XL-0807RGBC-WS2812B-S, U53 XL-0807RGBC-WS2812B-S, U54 XL-0807RGBC-WS2812B-S, U55 XL-0807RGBC-WS2812B-S, U56 XL-0807RGBC-WS2812B-S, U57 XL-0807RGBC-WS2812B-S, U58 XL-0807RGBC-WS2812B-S, U59 XL-0807RGBC-WS2812B-S, U6 XL-0807RGBC-WS2812B-S, U60 XL-0807RGBC-WS2812B-S, U61 XL-0807RGBC-WS2812B-S, U62 XL-0807RGBC-WS2812B-S, U63 XL-0807RGBC-WS2812B-S, U64 XL-0807RGBC-WS2812B-S, U65 XL-0807RGBC-WS2812B-S, U66 XL-0807RGBC-WS2812B-S, U67 XL-0807RGBC-WS2812B-S, U68 XL-0807RGBC-WS2812B-S, U69 XL-0807RGBC-WS2812B-S, U7 XL-0807RGBC-WS2812B-S, U70 XL-0807RGBC-WS2812B-S, U71 XL-0807RGBC-WS2812B-S, U72 XL-0807RGBC-WS2812B-S, U73 XL-0807RGBC-WS2812B-S, U74 XL-0807RGBC-WS2812B-S, U75 XL-0807RGBC-WS2812B-S, U76 XL-0807RGBC-WS2812B-S, U77 XL-0807RGBC-WS2812B-S, U78 XL-0807RGBC-WS2812B-S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

Commit message: Fully routed
Parts:
- removed SW1, SW2: SW_Push, symbol Switch:SW_Push
- added JP1: SolderJumper_2_Bridged, Jumper:SolderJumper-2_P1.3mm_Bridged_RoundedPad1.0x1.5mm, symbol Jumper:SolderJumper_2_Bridged
- added SW1, SW2: SKTAACE010, easyeda2kicad:KEY-SMD_4P-L2.6-W1.6-P0.80-LS3.0, symbol easyeda2kicad:SKTAACE010
- added TP4: TestPoint, TestPoint:TestPoint_Pad_2.0x2.0mm, symbol Connector:TestPoint
- J2: footprint (none) -> Connector_Wire:SolderWire-0.1sqmm_1x03_P3.6mm_D0.4mm_OD1mm
- R1, R4: footprint (none) -> Resistor_SMD:R_0603_1608Metric
- TP1, TP2, TP3: footprint (none) -> TestPoint:TestPoint_Pad_2.0x2.0mm
Connections:
- net +5V: now also U78.4 (VDD)
- net 3V3: no longer D1.2 (A)
- net GND: now also U76.2 (GND), U77.2 (GND), U78.2 (GND), SW1.2, SW1.4, SW2.2, SW2.4, TP4.1
- net at U77.1 (DO): now also TP3.1
- net at U78.1 (DO): now also U11.3 (DI)
- net at U78.3 (DI): now also U10.1 (DO)
- net at J1.13 (HS_G): now also SW2.1, SW2.3
- net at U56.3 (DI): now also JP1.2 (B)
- net at U66.3 (DI): now also U65.1 (DO)
- net at U55.1 (DO): now also JP1.1 (A); no longer TP3.1
- net at U71.3 (DI): now also U70.1 (DO)
- net at J1.12 (HS_F): now also SW1.1, SW1.3
- net at U60.1 (DO): now also U61.3 (DI)
- net at L1.2, U1.1 (SW): now also D1.2 (A)
- net at U76.3 (DI): now also U75.1 (DO)
Other:
- moved on the sheet: C2, D1, L1, TP3, U11, U12, U78

Commit message: Add LCSC part numbers
Parts:
- C1, C2: LCSC Part (none) -> C86295
- R1: LCSC Part (none) -> C137684
- R4: LCSC Part (none) -> C14675
- U1: LCSC Part (none) -> C84817
Changed lines of the file:
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@@
 			)
 		)
+		(property "LCSC Part" "C86295"
+			(at 82.55 151.13 90)
+			(effects
+				(font
+					(size 1.27 1.27)
+				)
+				(hide yes)
+			)
+		)
 		(pin "1"
 		)
@@
 			)
 		)
+		(property "LCSC Part" "C86295"
+			(at 58.42 137.16 0)
+			(effects
+				(font
+					(size 1.27 1.27)
+				)
+				(hide yes)
+			)
+		)
 		(pin "1"
 		)
@@
 			)
 		)
+		(property "LCSC Part" "C14675"
+			(at 82.55 146.05 90)
+			(effects
+				(font
+					(size 1.27 1.27)
+				)
+				(hide yes)
+			)
+		)
 		(pin "1"
 		)
@@
 			)
 		)
+		(property "LCSC Part" "C137684"
+			(at 92.71 146.05 90)
+			(effects
+				(font
+					(size 1.27 1.27)
+				)
+				(hide yes)
+			)
+		)
 		(pin "2"
 		)
@@
 			(at 74.93 134.62 0)
 			(effects
+				(font
+					(size 1.27 1.27)
+				)
+				(hide yes)
+			)
+		)
+		(property "LCSC Part" "C84817"
+			(at 74.93 134.62 0)
+			(effects

Commit message: Ready to fab
Other:
- note added: "<- Great Britain"
- note added: "Ireland ->"
- moved on the sheet: J2
Changed lines of the file:
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@@
 	(generator_version "9.0")
 	(paper "A4")
+	(text "<- Great Britain"
+		(exclude_from_sim no)
+		(at 1077.468 150.114 0)
+		(effects
+			(font
+				(size 1.27 1.27)
+			)
+		)
+	)
+	(text "Ireland ->"
+		(exclude_from_sim no)
+		(at 1102.36 149.86 0)
+		(effects
+			(font
+				(size 1.27 1.27)
+			)
+		)
+	)
 	(junction
 		(at 488.95 90.17)
@@
 	(wire
 		(pts
-			(xy 152.4 86.36) (xy 144.78 86.36)
+			(xy 181.61 83.82) (xy 173.99 83.82)
 		)
 		(stroke
@@
 	(wire
 		(pts
+			(xy 97.79 85.09) (xy 96.52 85.09)
+		)
+		(stroke
+			(width 0)
+			(type default)
+		)
+	)
+	(wire
+		(pts
 			(xy 765.81 67.31) (xy 783.59 67.31)
 		)
@@
 	(wire
 		(pts
-			(xy 157.48 88.9) (xy 144.78 88.9)
+			(xy 186.69 86.36) (xy 173.99 86.36)
 		)
 		(stroke
@@
 	(wire
 		(pts
+			(xy 97.79 82.55) (xy 96.52 82.55)
+		)
+		(stroke
+			(width 0)
+			(type default)
+		)
+	)
+	(wire
+		(pts
 			(xy 1356.36 71.12) (xy 1374.14 71.12)
 		)
@@
 	(wire
 		(pts
-			(xy 165.1 91.44) (xy 144.78 91.44)
+			(xy 194.31 88.9) (xy 173.99 88.9)
 		)
 		(stroke
@@
 	)
 	(label "HS_I"
-		(at 157.48 88.9 0)
+		(at 186.69 86.36 0)
 		(effects
 			(font
@@
 	)
 	(label "HS_I"
-		(at 96.52 85.09 0)
+		(at 97.79 85.09 0)
 		(effects
 			(font
@@
 	)
 	(label "GND"
-		(at 152.4 86.36 0)
+		(at 181.61 83.82 0)
 		(effects
 			(font
@@
 	)
 	(label "HS_H"
-		(at 96.52 82.55 0)
+		(at 97.79 82.55 0)
 		(effects
 			(font
@@
 	(symbol
 		(lib_id "power:+5V")
-		(at 165.1 91.44 0)
+		(at 194.31 88.9 0)
 		(unit 1)
 		(exclude_from_sim no)
@@
 		(dnp no)
 		(property "Reference" "#PWR064"
-			(at 165.1 95.25 0)
+			(at 194.31 92.71 0)
 			(effects
 				(font
@@
 		)
 		(property "Value" "+5V"
-			(at 167.64 91.186 0)
+			(at 196.85 88.646 0)
 			(effects
 				(font
@@
 		)
 		(property "Footprint" ""
-			(at 165.1 91.44 0)
+			(at 194.31 88.9 0)
 			(effects
 				(font
@@
 		)
 		(property "Datasheet" ""
-			(at 165.1 91.44 0)
+			(at 194.31 88.9 0)
 			(effects
 				(font
@@
 		)
 		(property "Description" "Power symbol creates a global label with name \"+5V\""
-			(at 165.1 91.44 0)
+			(at 194.31 88.9 0)
 			(effects
 				(font
@@
 	(symbol
 		(lib_id "Connector:Conn_01x03_Pin")
-		(at 139.7 88.9 0)
+		(at 168.91 86.36 0)
 		(unit 1)
 		(exclude_from_sim no)
@@
 		(fields_autoplaced yes)
 		(property "Reference" "J2"
-			(at 140.335 81.28 0)
+			(at 169.545 78.74 0)
 			(effects
 				(font
@@
 		)
 		(property "Value" "Conn_01x03_Pin"
-			(at 140.335 83.82 0)
+			(at 169.545 81.28 0)
 			(effects
 				(font
@@
 		)
 		(property "Footprint" "Connector_Wire:SolderWire-0.1sqmm_1x03_P3.6mm_D0.4mm_OD1mm"
-			(at 139.7 88.9 0)
+			(at 168.91 86.36 0)
 			(effects
 				(font
@@
 		)
 		(property "Datasheet" "~"
-			(at 139.7 88.9 0)
+			(at 168.91 86.36 0)
 			(effects
 				(font
@@
 		)
 		(property "Description" "Generic connector, single row, 01x03, script generated"
-			(at 139.7 88.9 0)
+			(at 168.91 86.36 0)
 			(effects
 				(font
@@
 	(sheet
 		(at 416.56 33.02)
-		(size 867.41 162.56)
+		(size 1033.78 163.83)
 		(exclude_from_sim no)
 		(in_bom yes)
@@
 		)
 		(property "Sheetfile" "untitled.kicad_sch"
-			(at 416.56 196.1646 0)
+			(at 416.56 197.4346 0)
 			(effects
 				(font
